File: lna/lna.kicad_sch (KiCad schematic)
At the start: 0 parts

Commit message: Start LNA project
Parts:
- added C1: 47pF, symbol Device:C
- added C2: 1.2pF, symbol Device:C
- added C3, C5: 0.01uF, symbol Device:C
- added C4: 330pF, symbol Device:C
- added J1: Conn_Coaxial, symbol Connector:Conn_Coaxial
- added J2: V5-GND, symbol lna_library:V5-GND
- added L1: 3nH, symbol Device:L
- added L2: 120nH, symbol Device:L
- added L3: 620nH, symbol Device:L
- added R1: 150R, symbol Device:R
- added U1: PGA-103+, Package_TO_SOT_SMD:SOT-89-3, symbol lna_library:PGA-103+
Connections:
- new net: C1.1, C2.1, J1.2 (Ext), L1.1
- new net: L3.2, R1.1
- new net: C4.1, R1.2
- new net: C2.2, L2.1
- new net: C3.1, L2.2
- new net: C3.2, L3.1, U1.1
- new net: C5.1, U1.3
- new net 5V: J2.2 (5V)
- new net GND: C1.2, C4.2, J1.1 (In), J2.1 (GND), L1.2, U1.2 (GND)
Other:
- note added: "Filter"
- title: (none) -> LNA + Filter 400-440 Mhz
