File: lna/lna.kicad_pcb (KiCad board)
At the start: 2 copper layers, 40 x 20 mm, 22 parts, among them J1 Conn_Coaxial, J2 V5-GND, J3 Conn_Coaxial, U1 PGA-103+

Commit message: Add so many holes
Routing:
- net GND: vias 8 -> 55
Changed lines of the file:
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@@
   )
   (dimension (type aligned) (layer "Dwgs.User")
-    (pts (xy 144.99971 84.99983) (xy 144.99971 104.99979))
+    (pts (xy 144.99971 85.29983) (xy 144.99971 105.29979))
     (height 0)
-    (gr_text "20.0000 mm" (at 143.84971 94.99981 270) (layer "Dwgs.User")
+    (gr_text "20.0000 mm" (at 143.84971 95.29981 270) (layer "Dwgs.User")
       (effects (font (size 1 1) (thickness 0.15)))
     )
@@
   (segment (start 143.5 90) (end 145 91.5) (width 1) (layer "F.Cu") (net 1))
   (segment (start 143.5 87) (end 143.5 90) (width 1) (layer "F.Cu") (net 1))
+  (via (at 137 103) (size 0.8) (drill 0.4) (layers "F.Cu" "B.Cu") (net 1))
+  (via (at 162 103) (size 0.8) (drill 0.4) (layers "F.Cu" "B.Cu") (net 1))
+  (via (at 149 97.3) (size 0.8) (drill 0.4) (layers "F.Cu" "B.Cu") (net 1))
+  (via (at 134 87) (size 0.8) (drill 0.4) (layers "F.Cu" "B.Cu") (net 1))
+  (via (at 149 103) (size 0.8) (drill 0.4) (layers "F.Cu" "B.Cu") (net 1))
+  (via (at 158 103) (size 0.8) (drill 0.4) (layers "F.Cu" "B.Cu") (net 1))
+  (via (at 140 97.3) (size 0.8) (drill 0.4) (layers "F.Cu" "B.Cu") (net 1))
+  (via (at 148 90) (size 0.8) (drill 0.4) (layers "F.Cu" "B.Cu") (net 1))
+  (via (at 137 87) (size 0.8) (drill 0.4) (layers "F.Cu" "B.Cu") (net 1))
+  (via (at 134 97.3) (size 0.8) (drill 0.4) (layers "F.Cu" "B.Cu") (net 1))
   (via (at 157.275 89) (size 0.8) (drill 0.4) (layers "F.Cu" "B.Cu") (net 1))
+  (via (at 137 90) (size 0.8) (drill 0.4) (layers "F.Cu" "B.Cu") (net 1))
+  (via (at 131 87) (size 0.8) (drill 0.4) (layers "F.Cu" "B.Cu") (net 1))
+  (via (at 151 90) (size 0.8) (drill 0.4) (layers "F.Cu" "B.Cu") (net 1))
+  (via (at 134 92) (size 0.8) (drill 0.4) (layers "F.Cu" "B.Cu") (net 1))
+  (via (at 156 92) (size 0.8) (drill 0.4) (layers "F.Cu" "B.Cu") (net 1))
   (via (at 145 94.8625) (size 0.8) (drill 0.4) (layers "F.Cu" "B.Cu") (net 1))
-  (via (at 128 90.5) (size 0.8) (drill 0.4) (layers "F.Cu" "B.Cu") (net 1))
+  (via (at 128 90) (size 0.8) (drill 0.4) (layers "F.Cu" "B.Cu") (net 1))
+  (via (at 137 92) (size 0.8) (drill 0.4) (layers "F.Cu" "B.Cu") (net 1))
+  (via (at 131 90) (size 0.8) (drill 0.4) (layers "F.Cu" "B.Cu") (net 1))
+  (via (at 146 97.3) (size 0.8) (drill 0.4) (layers "F.Cu" "B.Cu") (net 1))
+  (via (at 143 103) (size 0.8) (drill 0.4) (layers "F.Cu" "B.Cu") (net 1))
+  (via (at 131 100) (size 0.8) (drill 0.4) (layers "F.Cu" "B.Cu") (net 1))
+  (via (at 131 103) (size 0.8) (drill 0.4) (layers "F.Cu" "B.Cu") (net 1))
+  (via (at 134 103) (size 0.8) (drill 0.4) (layers "F.Cu" "B.Cu") (net 1))
+  (via (at 137 97.3) (size 0.8) (drill 0.4) (layers "F.Cu" "B.Cu") (net 1))
+  (via (at 158 97.3) (size 0.8) (drill 0.4) (layers "F.Cu" "B.Cu") (net 1))
   (via (at 151.2 100.2) (size 0.8) (drill 0.4) (layers "F.Cu" "B.Cu") (net 1))
+  (via (at 155 103) (size 0.8) (drill 0.4) (layers "F.Cu" "B.Cu") (net 1))
+  (via (at 148 92) (size 0.8) (drill 0.4) (layers "F.Cu" "B.Cu") (net 1))
+  (via (at 134 100) (size 0.8) (drill 0.4) (layers "F.Cu" "B.Cu") (net 1))
+  (via (at 159 90) (size 0.8) (drill 0.4) (layers "F.Cu" "B.Cu") (net 1))
   (via (at 157.275 90.8) (size 0.8) (drill 0.4) (layers "F.Cu" "B.Cu") (net 1))
-  (via (at 162 99.5) (size 0.8) (drill 0.4) (layers "F.Cu" "B.Cu") (net 1))
-  (via (at 162 90.5) (size 0.8) (drill 0.4) (layers "F.Cu" "B.Cu") (net 1))
-  (via (at 128 99.5) (size 0.8) (drill 0.4) (layers "F.Cu" "B.Cu") (net 1))
+  (via (at 140 92) (size 0.8) (drill 0.4) (layers "F.Cu" "B.Cu") (net 1))
+  (via (at 140 100) (size 0.8) (drill 0.4) (layers "F.Cu" "B.Cu") (net 1))
+  (via (at 159 92) (size 0.8) (drill 0.4) (layers "F.Cu" "B.Cu") (net 1))
+  (via (at 159 87) (size 0.8) (drill 0.4) (layers "F.Cu" "B.Cu") (net 1))
+  (via (at 128 103) (size 0.8) (drill 0.4) (layers "F.Cu" "B.Cu") (net 1))
+  (via (at 146 103) (size 0.8) (drill 0.4) (layers "F.Cu" "B.Cu") (net 1))
+  (via (at 162 100) (size 0.8) (drill 0.4) (layers "F.Cu" "B.Cu") (net 1))
+  (via (at 152 103) (size 0.8) (drill 0.4) (layers "F.Cu" "B.Cu") (net 1))
+  (via (at 162 87) (size 0.8) (drill 0.4) (layers "F.Cu" "B.Cu") (net 1))
+  (via (at 158 100) (size 0.8) (drill 0.4) (layers "F.Cu" "B.Cu") (net 1))
+  (via (at 155 97.3) (size 0.8) (drill 0.4) (layers "F.Cu" "B.Cu") (net 1))
+  (via (at 140 103) (size 0.8) (drill 0.4) (layers "F.Cu" "B.Cu") (net 1))
+  (via (at 162 90) (size 0.8) (drill 0.4) (layers "F.Cu" "B.Cu") (net 1))
+  (via (at 155 100) (size 0.8) (drill 0.4) (layers "F.Cu" "B.Cu") (net 1))
+  (via (at 128 87) (size 0.8) (drill 0.4) (layers "F.Cu" "B.Cu") (net 1))
+  (via (at 143 97.3) (size 0.8) (drill 0.4) (layers "F.Cu" "B.Cu") (net 1))
+  (via (at 137 100) (size 0.8) (drill 0.4) (layers "F.Cu" "B.Cu") (net 1))
+  (via (at 140 90) (size 0.8) (drill 0.4) (layers "F.Cu" "B.Cu") (net 1))
+  (via (at 134 90) (size 0.8) (drill 0.4) (layers "F.Cu" "B.Cu") (net 1))
+  (via (at 128 100) (size 0.8) (drill 0.4) (layers "F.Cu" "B.Cu") (net 1))
+  (via (at 152 97.3) (size 0.8) (drill 0.4) (layers "F.Cu" "B.Cu") (net 1))
+  (via (at 140 87) (size 0.8) (drill 0.4) (layers "F.Cu" "B.Cu") (net 1))
   (segment (start 128 90.75) (end 128 90.5) (width 1) (layer "B.Cu") (net 1))
   (segment (start 162 99.25) (end 162 90.75) (width 1) (layer "B.Cu") (net 1))
@@
   (segment (start 153.8875 90.8) (end 153.5375 90.8) (width 1) (layer "F.Cu") (net 6))
   (segment (start 154.45 86.8) (end 153.6875 86.8) (width 1) (layer "F.Cu") (net 6))
-  (segment (start 154.8875 95) (end 162 95) (width 3) (layer "F.Cu") (net 7))
+  (segment (start 154.8875 95) (end 160 95) (width 3) (layer "F.Cu") (net 7))
+  (segment (start 160 95) (end 162 95) (width 3) (layer "F.Cu") (net 7))
   (segment (start 152.1625 94.95) (end 152.2125 95) (width 1) (layer "F.Cu") (net 8))
   (segment (start 147.8 94.95) (end 147.089964 94.95) (width 1) (layer "F.Cu") (net 8))
