File: lna/lna.kicad_pcb (KiCad board)
At the start: 2 copper layers, 40 x 20 mm, 22 parts, among them J1 Conn_Coaxial, J2 V5-GND, J3 Conn_Coaxial, U1 PGA-103+

Commit message: V2
Parts:
- J1, J3: footprint Connector_Coaxial:SMA_Amphenol_132289_EdgeMount -> kp_labs:poprawione_sma
- moved G*** 2.55 mm to (158.2, 103.0)
- moved G*** 2.50 mm to (139.0, 103.0)
- moved L5 2.26 mm to (150.2, 94.2), turned to 90 degrees
- moved J1 2.21 mm to (130.2, 94.8)
- moved J3 2.20 mm to (159.8, 95.0)
- moved C3 2.10 mm to (148.3, 98.3)
- moved C4 2.03 mm to (153.2, 92.2)
- moved C5 2.03 mm to (153.2, 90.4)
- moved R1 1.98 mm to (145.2, 98.3)
- moved L4 1.91 mm to (142.0, 98.3)
- moved C1 1.76 mm to (134.3, 92.5)
- moved L1 1.76 mm to (134.3, 97.5)
- moved L3 1.69 mm to (140.9, 95.6)
- moved C6 1.41 mm to (154.8, 87.8)
- moved U1 0.72 mm to (144.4, 92.9)
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Routing:
- net Net-(L2-Pad1): track 2.08 -> 3.95 mm
- net Net-(C7-Pad2): track 7.11 -> 5.48 mm
- net Net-(C1-Pad1): track 6.24 -> 7.40 mm
- net Net-(C2-Pad2): track 0.48 -> 1.56 mm
- net Net-(C7-Pad1): track 7.91 -> 7.26 mm
Other:
- board size 40 x 20 mm -> 35 x 20 mm
- board text added: "V.2"

Commit message: Cleanup
Parts:
- J1, J3: footprint kp_labs:poprawione_sma -> fixed_sma:poprawione_sma
